Commit message: Second Commit

File: urdf/mark1.xacro (robot description, xacro)
@@ -143,10 +143,10 @@
         </inertial>
     </link>
-    <joint name="joint_3" type="fixed">
+    <joint name="joint_3" type="revolute">
         <origin rpy="0 0 0" xyz="0.1493 0.0 -0.089"/>
         <parent link="right_leg_rocker"/>
         <child link="right_leg_boogie"/>
         <axis xyz="0.0 1.0 0.0"/>
-        <limit lower="-0.523" upper="0.523" effort="1.0" velocity="1.0"/>
+        <limit lower="-0.523" upper="0.523" effort="1.0" velocity="0.5"/>
     </joint>
     <link name="right_leg_boogie">
@@ -199,10 +199,10 @@
         </inertial>
     </link>
-    <joint name="joint_4" type="fixed">
+    <joint name="joint_4" type="revolute">
         <origin rpy="0 0 0" xyz="0.1493 0.0 -0.089"/>
         <parent link="left_leg_rocker"/>
         <child link="left_leg_boogie"/>
         <axis xyz="0.0 1.0 0.0"/>
-        <limit lower="-0.523" upper="0.523" effort="1.0" velocity="1.0"/>
+        <limit lower="-0.523" upper="0.523" effort="1.0" velocity="0.5"/>
     </joint>
     <link name="left_leg_boogie">
@@ -260,5 +260,5 @@
         <child link="right_wheel_front"/>
         <axis xyz="0.0 1.0 0.0"/>
-        <limit effort="100.0" velocity="15.0"/>
+        <limit effort="1000.0" velocity="150.0"/>
     </joint>
     <link name="right_wheel_front">
@@ -290,5 +290,5 @@
         <child link="right_wheel_medium"/>
         <axis xyz="0.0 1.0 0.0"/>
-        <limit effort="100.0" velocity="15.0"/>
+        <limit effort="1000.0" velocity="150.0"/>
     </joint>
     <link name="right_wheel_medium">
@@ -320,5 +320,5 @@
         <child link="right_wheel_back"/>
         <axis xyz="0.0 1.0 0.0"/>
-        <limit effort="100.0" velocity="15.0"/>
+        <limit effort="1000.0" velocity="150.0"/>
     </joint>
     <link name="right_wheel_back">
@@ -350,5 +350,5 @@
         <child link="left_wheel_front"/>
         <axis xyz="0.0 1.0 0.0"/>
-        <limit effort="100.0" velocity="15.0"/>
+        <limit effort="1000.0" velocity="150.0"/>
     </joint>
     <link name="left_wheel_front">
@@ -380,5 +380,5 @@
         <child link="left_wheel_medium"/>
         <axis xyz="0.0 1.0 0.0"/>
-        <limit effort="100.0" velocity="15.0"/>
+        <limit effort="1000.0" velocity="150.0"/>
     </joint>
     <link name="left_wheel_medium">
@@ -410,5 +410,5 @@
         <child link="left_wheel_back"/>
         <axis xyz="0.0 1.0 0.0"/>
-        <limit effort="100.0" velocity="15.0"/>
+        <limit effort="1000.0" velocity="150.0"/>
     </joint>
     <link name="left_wheel_back">
@@ -540,16 +540,4 @@
         </inertial>
     </link>
-    <!-- 6Ruedas
-    <gazebo>
-      <plugin name="force_based_move_controller" filename="libgazebo_ros_force_based_move.so">
-        <commandTopic>/cmd_vel_raw</commandTopic>
-        <odometryTopic>odom</odometryTopic>
-        <odometryFrame>odom</odometryFrame>
-        <odometryRate>20.0</odometryRate>
-        <robotBaseFrame>chassis</robotBaseFrame>
-        <yaw_velocity_p_gain>250</yaw_velocity_p_gain>
-        <publishOdometryTf>1</publishOdometryTf>
-      </plugin>
-    </gazebo> -->
     <!-- Transmission -->
     <transmission name="tran1">
@@ -694,4 +682,17 @@
         </sensor>
     </gazebo>
+    <!-- Odom -->
+    <gazebo>
+        <plugin name="p3d_base_controller" filename="libgazebo_ros_p3d.so">
+            <alwaysOn>true</alwaysOn>
+            <updateRate>50.0</updateRate>
+            <bodyName>base_footprint</bodyName>
+            <topicName>odom</topicName>
+            <gaussianNoise>0.01</gaussianNoise>
+            <frameName>world</frameName>
+            <xyzOffsets>0 0 0</xyzOffsets>
+            <rpyOffsets>0 0 0</rpyOffsets>
+        </plugin>
+    </gazebo>
     <!-- Color -->
     <gazebo reference="chassis">
